Commit message: feat: enable continuous rotation for motor testbench
- Updated 'rotor_joint' from revolute to continuous type in motor_testbench.xacro
- Removed mechanical joint limits (lower/upper) to allow infinite rotation
- Exposed 'velocity' command interface in ros2_control.xacro
- Removed position command limits to support unrestricted tracking

File: src/gazebo_sim/gazebo_core/core_description/urdf/motor_testbench/modules/motor_testbench.xacro (robot description, xacro)
@@ -90,10 +90,10 @@
   </joint>
   <!-- Joint from base_link to rotor_link -->
-  <joint name="rotor_joint" type="revolute">
+  <joint name="rotor_joint" type="continuous">
     <origin xyz="0.0191322 0 0.101362" rpy="1.5708 -0 1.5708"/>
     <parent link="base_link"/>
     <child link="rotor_link"/>
     <axis xyz="0 0 1"/>
-    <limit effort="10" velocity="10" lower="-3.141592653589793" upper="3.141592653589793"/>
+    <limit effort="10" velocity="10"/>
   </joint>
 </robot>

File: src/gazebo_sim/gazebo_core/core_description/urdf/motor_testbench/modules/ros2_control.xacro (robot description, xacro)
@@ -6,8 +6,7 @@
     </hardware>
     <joint name="rotor_joint">
-      <command_interface name="position">
-        <param name="min">-1.57</param>
-        <param name="max">1.57</param>
-      </command_interface>
+      <command_interface name="position"/>
+      <!-- Add this new line to expose the velocity command -->
+      <command_interface name="velocity"/>
       <state_interface name="position"/>
       <state_interface name="velocity"/>

Commit message: fix: corrected rotor orientation

File: src/gazebo_sim/gazebo_core/core_description/urdf/motor_testbench/modules/motor_testbench.xacro (robot description, xacro)
@@ -91,5 +91,5 @@
   <!-- Joint from base_link to rotor_link -->
   <joint name="rotor_joint" type="continuous">
-    <origin xyz="0.0191322 0 0.101362" rpy="1.5708 -0 1.5708"/>
+    <origin xyz="0.0191322 0 0.101362" rpy="1.5708 1.5708 1.5708"/>
     <parent link="base_link"/>
     <child link="rotor_link"/>
