Commit message: refactor(urdf): upgrade 2WD robot model with xacro property tags

File: src/gazebo_sim/gazebo_core/core_description/urdf/tutorial_robot/robot_2wd.urdf.xacro (robot description, xacro)
@@ -1,4 +1,11 @@
 <?xml version="1.0"?>
-<robot name="robot_2wd">
+<robot name="robot_2wd" xmlns:xacro="http://www.ros.org/wiki/xacro">
+    <xacro:property name="base_footprint_to_chassis_z" value="0.1"/>
+    <xacro:property name="base_length" value="0.6" />
+    <xacro:property name="base_width" value="0.4" />
+    <xacro:property name="base_height" value="0.2" />
+    <xacro:property name="wheel_radius" value="0.1" />
+    <xacro:property name="wheel_width" value="0.05" />
+    <xacro:property name="caster_radius" value="0.05" />
     <material name="blue">
         <color rgba="0 0 0.5 1" />
@@ -11,7 +18,7 @@
         <visual>
             <geometry>
-                <box size="0.6 0.4 0.2" />
+                <box size="${base_length} ${base_width} ${base_height}" />
             </geometry>
-            <origin xyz="0 0 0.1" rpy="0 0 0" />
+            <origin xyz="0 0 ${base_height/2}" rpy="0 0 0" />
             <material name="blue" />
         </visual>
@@ -20,7 +27,7 @@
         <visual>
             <geometry>
-                <cylinder radius="0.1" length="0.05" />
+                <cylinder radius="${wheel_radius}" length="${wheel_width}" />
             </geometry>
-            <origin xyz="0 0 0" rpy="1.5708 0 0" />
+            <origin xyz="0 0 0" rpy="${pi / 2} 0 0" />
             <material name="grey" />
         </visual>
@@ -29,7 +36,7 @@
         <visual>
             <geometry>
-                <cylinder radius="0.1" length="0.05" />
+                <cylinder radius="${wheel_radius}" length="${wheel_width}" />
             </geometry>
-            <origin xyz="0 0 0" rpy="1.5708 0 0" />
+            <origin xyz="0 0 0" rpy="${pi / 2} 0 0" />
             <material name="grey" />
         </visual>
@@ -38,5 +45,5 @@
         <visual>
             <geometry>
-                <sphere radius="0.05" />
+                <sphere radius="${caster_radius}" />
             </geometry>
             <origin xyz="0 0 0" rpy="0 0 0" />
@@ -47,10 +54,10 @@
         <parent link="base_footprint" />
         <child link="base_link" />
-        <origin xyz="0 0 0.1" rpy="0 0 0" />
+        <origin xyz="0 0 ${base_footprint_to_chassis_z}" rpy="0 0 0" />
     </joint>
     <joint name="base_right_wheel_joint" type="continuous">
         <parent link="base_link" />
         <child link="right_wheel_link" />
-        <origin xyz="-0.15 -0.225 0" rpy="0 0 0" />
+        <origin xyz="-${base_length/4} -${base_width/2 + wheel_width/2} 0" rpy="0 0 0" />
         <axis xyz="0 1 0" />
     </joint>
@@ -58,5 +65,5 @@
         <parent link="base_link" />
         <child link="left_wheel_link" />
-        <origin xyz="-0.15 0.225 0" rpy="0 0 0" />
+        <origin xyz="-${base_length/4} ${base_width/2 + wheel_width/2} 0" rpy="0 0 0" />
         <axis xyz="0 1 0" />
     </joint>
@@ -64,5 +71,5 @@
         <parent link="base_link" />
         <child link="caster_wheel_link" />
-        <origin xyz="0.2 0 -0.05" rpy="0 0 0" />
+        <origin xyz="${base_length/3} 0 -${caster_radius}" rpy="0 0 0" />
     </joint>
 </robot>

Commit message: Refactor wheel links to use xacro macro

File: src/gazebo_sim/gazebo_core/core_description/urdf/tutorial_robot/robot_2wd.urdf.xacro (robot description, xacro)
@@ -24,5 +24,18 @@
         </visual>
     </link>
-    <link name="right_wheel_link">
+    <xacro:macro name="wheel_link" params="wheel">
+        <link name="${wheel}_wheel_link">
+            <visual>
+                <geometry>
+                    <cylinder radius="${wheel_radius}" length="${wheel_width}" />
+                </geometry>
+                <origin xyz="0 0 0" rpy="${pi / 2} 0 0" />
+                <material name="grey" />
+            </visual>
+        </link>
+    </xacro:macro>
+    <xacro:wheel_link wheel="left"/>
+    <xacro:wheel_link wheel="right"/>
+    <!-- <link name="right_wheel_link">
         <visual>
             <geometry>
@@ -41,5 +54,5 @@
             <material name="grey" />
         </visual>
-    </link>
+    </link> -->
     <link name="caster_wheel_link">
         <visual>

Commit message: chore: remove commented-out unused wheel links from 2wd robot urdf

File: src/gazebo_sim/gazebo_core/core_description/urdf/tutorial_robot/robot_2wd.urdf.xacro (robot description, xacro)
@@ -37,22 +37,4 @@
     <xacro:wheel_link wheel="left"/>
     <xacro:wheel_link wheel="right"/>
-    <!-- <link name="right_wheel_link">
-        <visual>
-            <geometry>
-                <cylinder radius="${wheel_radius}" length="${wheel_width}" />
-            </geometry>
-            <origin xyz="0 0 0" rpy="${pi / 2} 0 0" />
-            <material name="grey" />
-        </visual>
-    </link>
-    <link name="left_wheel_link">
-        <visual>
-            <geometry>
-                <cylinder radius="${wheel_radius}" length="${wheel_width}" />
-            </geometry>
-            <origin xyz="0 0 0" rpy="${pi / 2} 0 0" />
-            <material name="grey" />
-        </visual>
-    </link> -->
     <link name="caster_wheel_link">
         <visual>

Commit message: refactor: modularize robot_2wd urdf into separate common properties and robot component files

File: src/gazebo_sim/gazebo_core/core_description/urdf/tutorial_robot/robot_2wd.urdf.xacro (robot description, xacro)
@@ -1,70 +1,5 @@
 <?xml version="1.0"?>
 <robot name="robot_2wd" xmlns:xacro="http://www.ros.org/wiki/xacro">
-    <xacro:property name="base_footprint_to_chassis_z" value="0.1"/>
-    <xacro:property name="base_length" value="0.6" />
-    <xacro:property name="base_width" value="0.4" />
-    <xacro:property name="base_height" value="0.2" />
-    <xacro:property name="wheel_radius" value="0.1" />
-    <xacro:property name="wheel_width" value="0.05" />
-    <xacro:property name="caster_radius" value="0.05" />
-    <material name="blue">
-        <color rgba="0 0 0.5 1" />
-    </material>
-    <material name="grey">
-        <color rgba="0.4 0.4 0.5 1" />
-    </material>
-    <link name="base_footprint" />
-    <link name="base_link">
-        <visual>
-            <geometry>
-                <box size="${base_length} ${base_width} ${base_height}" />
-            </geometry>
-            <origin xyz="0 0 ${base_height/2}" rpy="0 0 0" />
-            <material name="blue" />
-        </visual>
-    </link>
-    <xacro:macro name="wheel_link" params="wheel">
-        <link name="${wheel}_wheel_link">
-            <visual>
-                <geometry>
-                    <cylinder radius="${wheel_radius}" length="${wheel_width}" />
-                </geometry>
-                <origin xyz="0 0 0" rpy="${pi / 2} 0 0" />
-                <material name="grey" />
-            </visual>
-        </link>
-    </xacro:macro>
-    <xacro:wheel_link wheel="left"/>
-    <xacro:wheel_link wheel="right"/>
-    <link name="caster_wheel_link">
-        <visual>
-            <geometry>
-                <sphere radius="${caster_radius}" />
-            </geometry>
-            <origin xyz="0 0 0" rpy="0 0 0" />
-            <material name="grey" />
-        </visual>
-    </link>
-    <joint name="base_footprint_joint" type="fixed">
-        <parent link="base_footprint" />
-        <child link="base_link" />
-        <origin xyz="0 0 ${base_footprint_to_chassis_z}" rpy="0 0 0" />
-    </joint>
-    <joint name="base_right_wheel_joint" type="continuous">
-        <parent link="base_link" />
-        <child link="right_wheel_link" />
-        <origin xyz="-${base_length/4} -${base_width/2 + wheel_width/2} 0" rpy="0 0 0" />
-        <axis xyz="0 1 0" />
-    </joint>
-    <joint name="base_left_wheel_joint" type="continuous">
-        <parent link="base_link" />
-        <child link="left_wheel_link" />
-        <origin xyz="-${base_length/4} ${base_width/2 + wheel_width/2} 0" rpy="0 0 0" />
-        <axis xyz="0 1 0" />
-    </joint>
-    <joint name="base_caster_wheel_joint" type="fixed">
-        <parent link="base_link" />
-        <child link="caster_wheel_link" />
-        <origin xyz="${base_length/3} 0 -${caster_radius}" rpy="0 0 0" />
-    </joint>
+    <xacro:include filename="$(find core_description)/urdf/tutorial_robot/modules/common_properties.xacro" />
+    <xacro:include filename="$(find core_description)/urdf/tutorial_robot/modules/robot_2wd.xacro" />
 </robot>
