Commit message: feat: add box_inertia macro and apply it to the robot base link

File: src/gazebo_sim/gazebo_core/core_description/urdf/tutorial_robot/modules/common_properties.xacro (robot description, xacro)
@@ -18,3 +18,12 @@
         </link>
     </xacro:macro>
+    <xacro:macro name="box_inertia" params="m x y z o_xyz o_rpy">
+        <inertial>
+            <mass value="${m}" />
+            <origin xyz="${o_xyz}" rpy="${o_rpy}" />
+            <inertia ixx="${(1.0/12.0) * m * (y*y + z*z)}" ixy="0" ixz="0"
+                     iyy="${(1.0/12.0) * m * (x*x + z*z)}" iyz="0"
+                     izz="${(1.0/12.0) * m * (x*x + y*y)}" />
+        </inertial>
+    </xacro:macro>
 </robot>

File: src/gazebo_sim/gazebo_core/core_description/urdf/tutorial_robot/modules/robot_2wd.xacro (robot description, xacro)
@@ -17,4 +17,7 @@
             <material name="blue" />
         </visual>
+        <xacro:box_inertia m="2.268"
+                           x="${base_length}" y="${base_width}" z="${base_height}"
+                           o_xyz="0 0 ${base_height/2}" o_rpy="0 0 0" />
     </link>
     <xacro:wheel_link wheel="left"/>

Commit message: feat: add cylinder and sphere inertia macros and apply to robot wheels and caster

File: src/gazebo_sim/gazebo_core/core_description/urdf/tutorial_robot/modules/common_properties.xacro (robot description, xacro)
@@ -16,4 +16,7 @@
                 <material name="grey" />
             </visual>
+            <xacro:cylinder_inertia m="0.854"
+                                    r="${wheel_radius}" h="${wheel_width}"
+                                    o_xyz="0 0 0" o_rpy="${pi / 2} 0 0" />
         </link>
     </xacro:macro>
@@ -27,3 +30,23 @@
         </inertial>
     </xacro:macro>
+    <xacro:macro name="cylinder_inertia" params="m r h o_xyz o_rpy">
+        <inertial>
+            <mass value="${m}"/>
+            <origin xyz="${o_xyz}" rpy="${o_rpy}"/>
+            <inertia
+                ixx="${(1.0/12.0) * m * (3 * r*r + h*h)}" ixy="0" ixz="0"
+                iyy="${(1.0/12.0) * m * (3 * r*r + h*h)}" iyz="0"
+                izz="${(1.0/2.0) * m * (r*r)}" />
+        </inertial>
+    </xacro:macro>
+    <xacro:macro name="sphere_inertia" params="m r o_xyz o_rpy">
+        <inertial>
+            <mass value="${m}" />
+            <origin xyz="${o_xyz}" rpy="${o_rpy}" />
+            <inertia
+                ixx="${(2.0/5.0) * m * (r*r)}" ixy="0" ixz="0"
+                iyy="${(2.0/5.0) * m * (r*r)}" iyz="0"
+                izz="${(2.0/5.0) * m * (r*r)}" />
+        </inertial>
+    </xacro:macro>
 </robot>

File: src/gazebo_sim/gazebo_core/core_description/urdf/tutorial_robot/modules/robot_2wd.xacro (robot description, xacro)
@@ -31,4 +31,5 @@
             <material name="grey" />
         </visual>
+        <xacro:sphere_inertia m="0.234" r="${caster_radius}" o_xyz="0 0 0" o_rpy="0 0 0" />
     </link>
     <joint name="base_footprint_joint" type="fixed">

Commit message: feat: add missing collision geometries to wheels, base, and caster links

File: src/gazebo_sim/gazebo_core/core_description/urdf/tutorial_robot/modules/common_properties.xacro (robot description, xacro)
@@ -16,4 +16,10 @@
                 <material name="grey" />
             </visual>
+            <collision>
+                <geometry>
+                    <sphere radius="${wheel_radius}" />
+                </geometry>
+                <origin xyz="0 0 0" rpy="${pi / 2} 0 0" />
+            </collision>
             <xacro:cylinder_inertia m="0.854"
                                     r="${wheel_radius}" h="${wheel_width}"

File: src/gazebo_sim/gazebo_core/core_description/urdf/tutorial_robot/modules/robot_2wd.xacro (robot description, xacro)
@@ -17,4 +17,10 @@
             <material name="blue" />
         </visual>
+        <collision>
+            <geometry>
+                <box size="${base_length} ${base_width} ${base_height}" />
+            </geometry>
+            <origin xyz="0 0 ${base_height/2}" rpy="0 0 0" />
+        </collision>
         <xacro:box_inertia m="2.268"
                            x="${base_length}" y="${base_width}" z="${base_height}"
@@ -31,4 +37,10 @@
             <material name="grey" />
         </visual>
+        <collision>
+            <geometry>
+                <sphere radius="${caster_radius}" />
+            </geometry>
+            <origin xyz="0 0 0" rpy="0 0 0" />
+        </collision>
         <xacro:sphere_inertia m="0.234" r="${caster_radius}" o_xyz="0 0 0" o_rpy="0 0 0" />
     </link>
