Commit message: feat: add optical frame and camera sensor configuration to robot URDF

File: src/gazebo_sim/gazebo_core/core_description/urdf/tutorial_robot/modules/camera.xacro (robot description, xacro)
@@ -21,4 +21,5 @@
         <xacro:box_inertia m="0.1" x="${camera_length}" y="${camera_width}" z="${camera_height}" o_xyz="${camera_length/2.0} 0 0" o_rpy="0 0 0" />
     </link>
+    <link name="camera_link_optical" />
     <joint name="camera_joint" type="fixed">
         <parent link="base_link" />
@@ -26,3 +27,35 @@
         <origin xyz="${base_length/2.0} 0 ${base_height/1.5}" rpy="0 0 0" />
     </joint>
+    <joint name="camera_optical_joint" type="fixed">
+        <origin xyz="0 0 0" rpy="${-pi/2} 0 ${-pi/2}"/>
+        <parent link="camera_link"/>
+        <child link="camera_link_optical"/>
+    </joint>
+    <gazebo reference="camera_link">
+        <sensor name="camera" type="camera">
+            <camera>
+                <horizontal_fov>1.3962634</horizontal_fov>
+                <image>
+                    <width>640</width>
+                    <height>480</height>
+                    <format>R8G8B8</format>
+                </image>
+                <clip>
+                    <near>0.1</near>
+                    <far>15</far>
+                </clip>
+                <noise>
+                    <type>gaussian</type>
+                    <mean>0.0</mean>
+                    <stddev>0.007</stddev>
+                </noise>
+                <optical_frame_id>camera_link_optical</optical_frame_id>
+                <camera_info_topic>camera/camera_info</camera_info_topic>
+            </camera>
+            <always_on>1</always_on>
+            <update_rate>20</update_rate>
+            <visualize>true</visualize>
+            <topic>camera/image_raw</topic>
+        </sensor>
+    </gazebo>
 </robot>
