Commit message: refactor(core_description): implement optical frame pattern for lidar
- Decoupled the physical lidar visual/collision (`scan_link`) from the sensor optical origin.
- Added `scan_optical_frame` as an invisible, weightless dummy link representing the exact center of the laser array.
- Shifted physical body visual origin to cleanly mount on the chassis while preserving mathematical accuracy for the sensor.
- Updated Gazebo plugin to reference the new optical frame for correct TF tree resolution in RViz.

File: src/gazebo_sim/gazebo_core/core_description/urdf/tutorial_robot/modules/lidar.xacro (robot description, xacro)
@@ -3,4 +3,5 @@
     <xacro:property name="lidar_height" value="0.05" />
     <xacro:property name="lidar_radius" value="0.05" />
+    <!-- The physical lidar body -->
     <link name="scan_link">
         <visual>
@@ -8,5 +9,6 @@
                 <cylinder length="${lidar_height}" radius="${lidar_radius}" />
             </geometry>
-            <origin xyz="0 0 0" rpy="0 0 0" />
+            <!-- Offset visual so the bottom face sits on the joint -->
+            <origin xyz="0 0 ${lidar_height/2}" rpy="0 0 0" />
             <material name="grey" />
         </visual>
@@ -15,18 +17,29 @@
                 <cylinder length="${lidar_height}" radius="${lidar_radius}" />
             </geometry>
-            <origin xyz="0 0 0" rpy="0 0 0" />
+            <origin xyz="0 0 ${lidar_height/2}" rpy="0 0 0" />
         </collision>
     </link>
-    <joint name="lidar_joint" type="fixed">
+    <!-- Joint mounting the physical body to the chassis -->
+    <joint name="lidar_mount_joint" type="fixed">
         <parent link="base_link" />
         <child link="scan_link" />
-        <origin xyz="${base_length/4} 0 ${base_height + lidar_height/2}" rpy="0 0 0" />
+        <!-- Placed exactly on the roof of the base_link -->
+        <origin xyz="${base_length/4} 0 ${base_height}" rpy="0 0 0" />
+    </joint>
+    <!-- The fake link representing the optical center -->
+    <link name="scan_optical_frame" />
+    <!-- Joint placing the fake link at the mathematical center of the sensor -->
+    <joint name="lidar_optical_joint" type="fixed">
+        <parent link="scan_link" />
+        <child link="scan_optical_frame" />
+        <!-- Shifted up from the mount point to the center where lasers shoot -->
+        <origin xyz="0 0 ${lidar_height/2}" rpy="0 0 0" />
     </joint>
     <!-- refer https://sdformat.org/spec/1.12/sensor/ for sensors -->
-    <gazebo reference="scan_link">
+    <gazebo reference="scan_optical_frame">
         <sensor name="gpu_lidar" type="gpu_lidar">
-            <pose relative_to='scan_link'>0 0 0 0 0 0</pose>
+            <pose relative_to='scan_optical_frame'>0 0 0 0 0 0</pose>
             <topic>scan</topic>
-            <gz_frame_id>scan_link</gz_frame_id>
+            <gz_frame_id>scan_optical_frame</gz_frame_id>
             <update_rate>10</update_rate>
             <ray>
