Commit message: feat: improve URDF and integrate custom 3D meshes
- Updated URDF configurations to reference the newly improved mesh files

File: src/Odometry_and_Control/bumperbot_description/urdf/bumperbot.urdf.xacro (robot description, xacro)
@@ -1,6 +1,7 @@
-<?xml version="1.0"?>
+<?xml version="1.0" ?>
 <robot name="bumperbot" xmlns:xacro="http://ros.org/wiki/xacro">
-  <xacro:include filename="$(find bumperbot_description)/urdf/include/bumperbot_mobile_base.xacro"/>
-  <xacro:include filename="$(find bumperbot_description)/urdf/include/bumperbot.gazebo.xacro"/>
-  <xacro:include filename="$(find bumperbot_description)/urdf/include/bumperbot_ros2control.xacro"/>
+  <xacro:include filename="$(find bumperbot_description)/urdf/include/common_properties.xacro" />
+  <xacro:include filename="$(find bumperbot_description)/urdf/include/bumperbot_mobile_base.xacro" />
+  <xacro:include filename="$(find bumperbot_description)/urdf/include/bumperbot.gazebo.xacro" />
+  <xacro:include filename="$(find bumperbot_description)/urdf/include/bumperbot_ros2control.xacro" />
 </robot>

File: src/Odometry_and_Control/bumperbot_description/urdf/include/bumperbot_mobile_base.xacro (robot description, xacro)
@@ -1,139 +1,592 @@
-<?xml version="1.0"?>
+<?xml version="1.0" ?>
 <robot xmlns:xacro="http://ros.org/wiki/xacro">
+  <xacro:property name="base_footprint_to_base_link_z" value="0.00999676" />
+  <xacro:property name="mesh_format" value="gltf" />
   <link name="base_footprint"/>
+  <joint name="base_footprint_joint" type="fixed">
+    <parent link="base_footprint"/>
+    <child link="base_link"/>
+    <!-- <origin xyz="0 0 0"/> -->
+    <origin xyz="0 0 ${base_footprint_to_base_link_z}"/>
+  </joint>
+<!-- Link base_link -->
   <link name="base_link">
     <inertial>
-      <origin xyz="0 0 0.04" rpy="0.0 0.25 0.3" />
-      <mass value="8.2573504e-01"/>
-      <inertia ixx="2.2124416e-02" ixy="-1.2294101e-04" ixz="3.4938785e-04"
-               iyy="2.1193702e-02" iyz="-5.0120904e-05"
-               izz="2.0064271e-02" />
+      <origin xyz="-0.000500099 3.9e-11 0.0388508" rpy="0 0 0"/>
+      <mass value="0.427641"/>
+      <inertia ixx="0.000917472" ixy="-1.75126e-05" ixz="-6.25e-10" iyy="0.000910074" iyz="2e-12" izz="0.0011829"/>
     </inertial>
-    <visual>
-      <origin xyz="0 0 0" rpy="0 0 0" />
-      <geometry>
-        <mesh filename="package://bumperbot_description/meshes/base_link.gltf" />
-      </geometry>
-    </visual>
-    <collision>
-      <origin xyz="0 0 0" rpy="0 0 0" />
-      <geometry>
-        <mesh filename="package://bumperbot_description/meshes/base_link.gltf" />
+    <!-- Part spacer_hex -->
+    <visual>
+      <origin xyz="0.0635 -0.024 0.0434998" rpy="0 -0 -0"/>
+      <geometry>
+        <mesh filename="package://bumperbot_description/meshes/spacer_hex.${mesh_format}"/>
+      </geometry>
+      <material name="spacer_hex_material">
+        <color rgba="0.980392 0.796078 0.262745 1"/>
+      </material>
+    </visual>
+    <collision>
+      <origin xyz="0.0635 -0.024 0.0434998" rpy="0 -0 -0"/>
+      <geometry>
+        <mesh filename="package://bumperbot_description/meshes/spacer_hex.${mesh_format}"/>
+      </geometry>
+    </collision>
+    <!-- Part spacer_hex_2 -->
+    <visual>
+      <origin xyz="-0.0645 -0.012 0.0434998" rpy="0 -0 -0"/>
+      <geometry>
+        <mesh filename="package://bumperbot_description/meshes/spacer_hex.${mesh_format}"/>
+      </geometry>
+      <material name="spacer_hex_2_material">
+        <color rgba="0.980392 0.796078 0.262745 1"/>
+      </material>
+    </visual>
+    <collision>
+      <origin xyz="-0.0645 -0.012 0.0434998" rpy="0 -0 -0"/>
+      <geometry>
+        <mesh filename="package://bumperbot_description/meshes/spacer_hex.${mesh_format}"/>
+      </geometry>
+    </collision>
+    <!-- Part spacer_hex_3 -->
+    <visual>
+      <origin xyz="0.0635 0.012 0.0434998" rpy="0 0 -0"/>
+      <geometry>
+        <mesh filename="package://bumperbot_description/meshes/spacer_hex.${mesh_format}"/>
+      </geometry>
+      <material name="spacer_hex_3_material">
+        <color rgba="0.980392 0.796078 0.262745 1"/>
+      </material>
+    </visual>
+    <collision>
+      <origin xyz="0.0635 0.012 0.0434998" rpy="0 0 -0"/>
+      <geometry>
+        <mesh filename="package://bumperbot_description/meshes/spacer_hex.${mesh_format}"/>
+      </geometry>
+    </collision>
+    <!-- Part spacer_hex_4 -->
+    <visual>
+      <origin xyz="0.0235 0.064 0.0434998" rpy="0 -0 -1.5708"/>
+      <geometry>
+        <mesh filename="package://bumperbot_description/meshes/spacer_hex.${mesh_format}"/>
+      </geometry>
+      <material name="spacer_hex_4_material">
+        <color rgba="0.980392 0.796078 0.262745 1"/>
+      </material>
+    </visual>
+    <collision>
+      <origin xyz="0.0235 0.064 0.0434998" rpy="0 -0 -1.5708"/>
+      <geometry>
+        <mesh filename="package://bumperbot_description/meshes/spacer_hex.${mesh_format}"/>
+      </geometry>
+    </collision>
+    <!-- Part base_plate -->
+    <visual>
+      <origin xyz="-0.0005 -0 0.037" rpy="0 -0 1.5708"/>
+      <geometry>
+        <mesh filename="package://bumperbot_description/meshes/base_plate.${mesh_format}"/>
+      </geometry>
+      <material name="base_plate_material">
+        <color rgba="0.117647 0.117647 0.117647 1"/>
+      </material>
+    </visual>
+    <collision>
+      <origin xyz="-0.0005 -0 0.037" rpy="0 -0 1.5708"/>
+      <geometry>
+        <mesh filename="package://bumperbot_description/meshes/base_plate.${mesh_format}"/>
+      </geometry>
+    </collision>
+    <!-- Part spacer_hex_5 -->
+    <visual>
+      <origin xyz="-0.0645 0.024 0.0434998" rpy="-0 -0 -0"/>
+      <geometry>
+        <mesh filename="package://bumperbot_description/meshes/spacer_hex.${mesh_format}"/>
+      </geometry>
+      <material name="spacer_hex_5_material">
+        <color rgba="0.980392 0.796078 0.262745 1"/>
+      </material>
+    </visual>
+    <collision>
+      <origin xyz="-0.0645 0.024 0.0434998" rpy="-0 -0 -0"/>
+      <geometry>
+        <mesh filename="package://bumperbot_description/meshes/spacer_hex.${mesh_format}"/>
+      </geometry>
+    </collision>
+    <!-- Part spacer_hex_6 -->
+    <visual>
+      <origin xyz="-0.0245 -0.064 0.0434998" rpy="0 -0 1.5708"/>
+      <geometry>
+        <mesh filename="package://bumperbot_description/meshes/spacer_hex.${mesh_format}"/>
+      </geometry>
+      <material name="spacer_hex_6_material">
+        <color rgba="0.980392 0.796078 0.262745 1"/>
+      </material>
+    </visual>
+    <collision>
+      <origin xyz="-0.0245 -0.064 0.0434998" rpy="0 -0 1.5708"/>
+      <geometry>
+        <mesh filename="package://bumperbot_description/meshes/spacer_hex.${mesh_format}"/>
+      </geometry>
+    </collision>
+    <!-- Part base_plate_2 -->
+    <visual>
+      <origin xyz="-0.0005 -0 0.037" rpy="0 -0 -1.5708"/>
+      <geometry>
+        <mesh filename="package://bumperbot_description/meshes/base_plate.${mesh_format}"/>
+      </geometry>
+      <material name="base_plate_2_material">
+        <color rgba="0.117647 0.117647 0.117647 1"/>
+      </material>
+    </visual>
+    <collision>
+      <origin xyz="-0.0005 -0 0.037" rpy="0 -0 -1.5708"/>
+      <geometry>
+        <mesh filename="package://bumperbot_description/meshes/base_plate.${mesh_format}"/>
+      </geometry>
+    </collision>
+    <!-- Part base_plate_3 -->
+    <visual>
+      <origin xyz="-0.0005 -0 0.074" rpy="0 -0 1.5708"/>
+      <geometry>
+        <mesh filename="package://bumperbot_description/meshes/base_plate.${mesh_format}"/>
+      </geometry>
+      <material name="base_plate_3_material">
+        <color rgba="0.117647 0.117647 0.117647 1"/>
+      </material>
+    </visual>
+    <collision>
+      <origin xyz="-0.0005 -0 0.074" rpy="0 -0 1.5708"/>
+      <geometry>
+        <mesh filename="package://bumperbot_description/meshes/base_plate.${mesh_format}"/>
+      </geometry>
+    </collision>
+    <!-- Part base_plate_4 -->
+    <visual>
+      <origin xyz="-0.0005 -0 0.074" rpy="0 -0 -1.5708"/>
+      <geometry>
+        <mesh filename="package://bumperbot_description/meshes/base_plate.${mesh_format}"/>
+      </geometry>
+      <material name="base_plate_4_material">
+        <color rgba="0.117647 0.117647 0.117647 1"/>
+      </material>
+    </visual>
+    <collision>
+      <origin xyz="-0.0005 -0 0.074" rpy="0 -0 -1.5708"/>
+      <geometry>
+        <mesh filename="package://bumperbot_description/meshes/base_plate.${mesh_format}"/>
+      </geometry>
+    </collision>
+    <!-- Part spacer_hex_7 -->
+    <visual>
+      <origin xyz="0.0635 -0.024 0.0064998" rpy="0 -0 0"/>
+      <geometry>
+        <mesh filename="package://bumperbot_description/meshes/spacer_hex.${mesh_format}"/>
+      </geometry>
+      <material name="spacer_hex_7_material">
+        <color rgba="0.980392 0.796078 0.262745 1"/>
+      </material>
+    </visual>
+    <collision>
+      <origin xyz="0.0635 -0.024 0.0064998" rpy="0 -0 0"/>
+      <geometry>
+        <mesh filename="package://bumperbot_description/meshes/spacer_hex.${mesh_format}"/>
+      </geometry>
+    </collision>
+    <!-- Part motor_bracket_left -->
+    <visual>
+      <origin xyz="-0.0005 0.0482736 0.00899984" rpy="0 -0 0"/>
+      <geometry>
+        <mesh filename="package://bumperbot_description/meshes/motor_bracket_left.${mesh_format}"/>
+      </geometry>
+      <material name="motor_bracket_left_material">
+        <color rgba="0.262745 0.282353 0.301961 1"/>
+      </material>
+    </visual>
+    <collision>
+      <origin xyz="-0.0005 0.0482736 0.00899984" rpy="0 -0 0"/>
+      <geometry>
+        <mesh filename="package://bumperbot_description/meshes/motor_bracket_left.${mesh_format}"/>
+      </geometry>
+    </collision>
+    <!-- Part spacer_hex_8 -->
+    <visual>
+      <origin xyz="-0.0645 -0.012 0.0064998" rpy="0 -0 0"/>
+      <geometry>
+        <mesh filename="package://bumperbot_description/meshes/spacer_hex.${mesh_format}"/>
+      </geometry>
+      <material name="spacer_hex_8_material">
+        <color rgba="0.980392 0.796078 0.262745 1"/>
+      </material>
+    </visual>
+    <collision>
+      <origin xyz="-0.0645 -0.012 0.0064998" rpy="0 -0 0"/>
+      <geometry>
+        <mesh filename="package://bumperbot_description/meshes/spacer_hex.${mesh_format}"/>
+      </geometry>
+    </collision>
+    <!-- Part spacer_hex_9 -->
+    <visual>
+      <origin xyz="0.0635 0.012 0.0064998" rpy="0 0 0"/>
+      <geometry>
+        <mesh filename="package://bumperbot_description/meshes/spacer_hex.${mesh_format}"/>
+      </geometry>
+      <material name="spacer_hex_9_material">
+        <color rgba="0.980392 0.796078 0.262745 1"/>
+      </material>
+    </visual>
+    <collision>
+      <origin xyz="0.0635 0.012 0.0064998" rpy="0 0 0"/>
+      <geometry>
+        <mesh filename="package://bumperbot_description/meshes/spacer_hex.${mesh_format}"/>
+      </geometry>
+    </collision>
+    <!-- Part spacer_hex_10 -->
+    <visual>
+      <origin xyz="0.0235 0.064 0.0064998" rpy="0 -0 -1.5708"/>
+      <geometry>
+        <mesh filename="package://bumperbot_description/meshes/spacer_hex.${mesh_format}"/>
+      </geometry>
+      <material name="spacer_hex_10_material">
+        <color rgba="0.980392 0.796078 0.262745 1"/>
+      </material>
+    </visual>
+    <collision>
+      <origin xyz="0.0235 0.064 0.0064998" rpy="0 -0 -1.5708"/>
+      <geometry>
+        <mesh filename="package://bumperbot_description/meshes/spacer_hex.${mesh_format}"/>
+      </geometry>
+    </collision>
+    <!-- Part motor_bracket_right -->
+    <visual>
+      <origin xyz="-0.0005 -0.0482736 0.00899984" rpy="0 -0 0"/>
+      <geometry>
+        <mesh filename="package://bumperbot_description/meshes/motor_bracket_right.${mesh_format}"/>
+      </geometry>
+      <material name="motor_bracket_right_material">
+        <color rgba="0.262745 0.282353 0.301961 1"/>
+      </material>
+    </visual>
+    <collision>
+      <origin xyz="-0.0005 -0.0482736 0.00899984" rpy="0 -0 0"/>
+      <geometry>
+        <mesh filename="package://bumperbot_description/meshes/motor_bracket_right.${mesh_format}"/>
+      </geometry>
+    </collision>
+    <!-- Part actuatordc_left -->
+    <visual>
+      <origin xyz="-0.0005 0.0667736 0.0239998" rpy="-0 -0 0"/>
+      <geometry>
+        <mesh filename="package://bumperbot_description/meshes/actuatordc_left.${mesh_format}"/>
+      </geometry>
+      <material name="actuatordc_left_material">
+        <color rgba="0.647059 0.647059 0.647059 1"/>
+      </material>
+    </visual>
+    <collision>
+      <origin xyz="-0.0005 0.0667736 0.0239998" rpy="-0 -0 0"/>
+      <geometry>
+        <mesh filename="package://bumperbot_description/meshes/actuatordc_left.${mesh_format}"/>
+      </geometry>
+    </collision>
+    <!-- Part base_plate_5 -->
+    <visual>
+      <origin xyz="-0.0005 -0 0" rpy="0 -0 1.5708"/>
+      <geometry>
+        <mesh filename="package://bumperbot_description/meshes/base_plate.${mesh_format}"/>
+      </geometry>
+      <material name="base_plate_5_material">
+        <color rgba="0.117647 0.117647 0.117647 1"/>
+      </material>
+    </visual>
+    <collision>
+      <origin xyz="-0.0005 -0 0" rpy="0 -0 1.5708"/>
+      <geometry>
+        <mesh filename="package://bumperbot_description/meshes/base_plate.${mesh_format}"/>
+      </geometry>
+    </collision>
+    <!-- Part actuatordc_right -->
+    <visual>
+      <origin xyz="-0.0005 -0.0667736 0.0239998" rpy="0 0 0"/>
+      <geometry>
+        <mesh filename="package://bumperbot_description/meshes/actuatordc_right.${mesh_format}"/>
+      </geometry>
+      <material name="actuatordc_right_material">
+        <color rgba="0.647059 0.647059 0.647059 1"/>
+      </material>
+    </visual>
+    <collision>
+      <origin xyz="-0.0005 -0.0667736 0.0239998" rpy="0 0 0"/>
+      <geometry>
+        <mesh filename="package://bumperbot_description/meshes/actuatordc_right.${mesh_format}"/>
+      </geometry>
+    </collision>
+    <!-- Part spacer_hex_11 -->
+    <visual>
+      <origin xyz="-0.0645 0.024 0.0064998" rpy="-0 -0 0"/>
+      <geometry>
+        <mesh filename="package://bumperbot_description/meshes/spacer_hex.${mesh_format}"/>
+      </geometry>
+      <material name="spacer_hex_11_material">
+        <color rgba="0.980392 0.796078 0.262745 1"/>
+      </material>
+    </visual>
+    <collision>
+      <origin xyz="-0.0645 0.024 0.0064998" rpy="-0 -0 0"/>
+      <geometry>
+        <mesh filename="package://bumperbot_description/meshes/spacer_hex.${mesh_format}"/>
+      </geometry>
+    </collision>
+    <!-- Part spacer_hex_12 -->
+    <visual>
+      <origin xyz="-0.0245 -0.064 0.0064998" rpy="0 -0 1.5708"/>
+      <geometry>
+        <mesh filename="package://bumperbot_description/meshes/spacer_hex.${mesh_format}"/>
+      </geometry>
+      <material name="spacer_hex_12_material">
+        <color rgba="0.980392 0.796078 0.262745 1"/>
+      </material>
+    </visual>
+    <collision>
+      <origin xyz="-0.0245 -0.064 0.0064998" rpy="0 -0 1.5708"/>
+      <geometry>
+        <mesh filename="package://bumperbot_description/meshes/spacer_hex.${mesh_format}"/>
+      </geometry>
+    </collision>
+    <!-- Part base_plate_6 -->
+    <visual>
+      <origin xyz="-0.0005 -0 0" rpy="0 -0 -1.5708"/>
+      <geometry>
+        <mesh filename="package://bumperbot_description/meshes/base_plate.${mesh_format}"/>
+      </geometry>
+      <material name="base_plate_6_material">
+        <color rgba="0.117647 0.117647 0.117647 1"/>
+      </material>
+    </visual>
+    <collision>
+      <origin xyz="-0.0005 -0 0" rpy="0 -0 -1.5708"/>
+      <geometry>
+        <mesh filename="package://bumperbot_description/meshes/base_plate.${mesh_format}"/>
       </geometry>
     </collision>
   </link>
-  <joint name="base_joint" type="fixed">
-    <parent link="base_footprint"/>
-    <child link="base_link" />
-    <origin xyz="0 0 0.033" rpy="0 0 0"/>
+  <!-- Link caster_wheel -->
+  <link name="caster_wheel">
+    <inertial>
+      <origin xyz="1.49659e-07 1.68167e-07 0.000721256" rpy="0 0 0"/>
+      <mass value="0.00466009"/>
+      <inertia ixx="1.13552e-07" ixy="-5e-12" ixz="1e-12" iyy="7.7488e-08" iyz="1e-12" izz="1.35464e-07"/>
+    </inertial>
+    <!-- Part caster_ball -->
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