Commit message: refactor: replace STL meshes with GLTF in mobile base URDF
- The STL geometry files were swapped out for modern GLTF assets. GLTF retains
the material colors defined in the CAD model, allowing the robot’s visual
representation to display the intended colors automatically without
post‑processing textures.

File: src/Odometry_and_Control/bumperbot_description/urdf/include/bumperbot_mobile_base.xacro (robot description, xacro)
@@ -13,5 +13,5 @@
       <origin xyz="0 0 0" rpy="0 0 0" />
       <geometry>
-        <mesh filename="package://bumperbot_description/meshes/base_link.STL" />
+        <mesh filename="package://bumperbot_description/meshes/base_link.gltf" />
       </geometry>
     </visual>
@@ -19,5 +19,5 @@
       <origin xyz="0 0 0" rpy="0 0 0" />
       <geometry>
-        <mesh filename="package://bumperbot_description/meshes/base_link.STL" />
+        <mesh filename="package://bumperbot_description/meshes/base_link.gltf" />
       </geometry>
     </collision>
@@ -39,5 +39,5 @@
       <origin xyz="0 0 0" rpy="1.57 0 0" />
       <geometry>
-        <mesh filename="package://bumperbot_description/meshes/wheel_right_link.STL" />
+        <mesh filename="package://bumperbot_description/meshes/wheel_right_link.gltf" />
       </geometry>
     </visual>
@@ -67,5 +67,5 @@
       <origin xyz="0 0 0" rpy="-1.57 0 0" />
       <geometry>
-        <mesh filename="package://bumperbot_description/meshes/wheel_left_link.STL" />
+        <mesh filename="package://bumperbot_description/meshes/wheel_left_link.gltf" />
       </geometry>
     </visual>
@@ -94,5 +94,5 @@
       <origin xyz="0 0 0" rpy="0 0 0" />
       <geometry>
-        <mesh filename="package://bumperbot_description/meshes/caster_front_link.STL" />
+        <mesh filename="package://bumperbot_description/meshes/caster_front_link.gltf" />
       </geometry>
     </visual>
@@ -121,5 +121,5 @@
       <origin xyz="0 0 0" rpy="0 0 0" />
       <geometry>
-        <mesh filename="package://bumperbot_description/meshes/caster_rear_link.STL" />
+        <mesh filename="package://bumperbot_description/meshes/caster_rear_link.gltf" />
       </geometry>
     </visual>

Commit message: feat: add L298N motor driver mesh and raspberry pi 5 to the URDF model.

File: src/Odometry_and_Control/bumperbot_description/urdf/include/bumperbot_mobile_base.xacro (robot description, xacro)
@@ -81,5 +81,5 @@
       </geometry>
     </collision>
-    <!-- Part base_plate -->
+    <!-- Part base_plate_mid_left -->
     <visual>
       <origin xyz="-0.0005 -0 0.037" rpy="0 -0 1.5708"/>
@@ -87,5 +87,5 @@
         <mesh filename="package://bumperbot_description/meshes/base_plate.${mesh_format}"/>
       </geometry>
-      <material name="base_plate_material">
+      <material name="base_plate_mid_left_material">
         <color rgba="0.117647 0.117647 0.117647 1"/>
       </material>
@@ -129,5 +129,5 @@
       </geometry>
     </collision>
-    <!-- Part base_plate_2 -->
+    <!-- Part base_plate_mid_right -->
     <visual>
       <origin xyz="-0.0005 -0 0.037" rpy="0 -0 -1.5708"/>
@@ -135,5 +135,5 @@
         <mesh filename="package://bumperbot_description/meshes/base_plate.${mesh_format}"/>
       </geometry>
-      <material name="base_plate_2_material">
+      <material name="base_plate_mid_right_material">
         <color rgba="0.117647 0.117647 0.117647 1"/>
       </material>
@@ -145,5 +145,5 @@
       </geometry>
     </collision>
-    <!-- Part base_plate_3 -->
+    <!-- Part base_plate_top_left -->
     <visual>
       <origin xyz="-0.0005 -0 0.074" rpy="0 -0 1.5708"/>
@@ -151,5 +151,5 @@
         <mesh filename="package://bumperbot_description/meshes/base_plate.${mesh_format}"/>
       </geometry>
-      <material name="base_plate_3_material">
+      <material name="base_plate_top_left_material">
         <color rgba="0.117647 0.117647 0.117647 1"/>
       </material>
@@ -161,5 +161,5 @@
       </geometry>
     </collision>
-    <!-- Part base_plate_4 -->
+    <!-- Part base_plate_top_right -->
     <visual>
       <origin xyz="-0.0005 -0 0.074" rpy="0 -0 -1.5708"/>
@@ -167,5 +167,5 @@
         <mesh filename="package://bumperbot_description/meshes/base_plate.${mesh_format}"/>
       </geometry>
-      <material name="base_plate_4_material">
+      <material name="base_plate_top_right_material">
         <color rgba="0.117647 0.117647 0.117647 1"/>
       </material>
@@ -289,5 +289,5 @@
       </geometry>
     </collision>
-    <!-- Part base_plate_5 -->
+    <!-- Part base_plate_bottom_left -->
     <visual>
       <origin xyz="-0.0005 -0 0" rpy="0 -0 1.5708"/>
@@ -295,5 +295,5 @@
         <mesh filename="package://bumperbot_description/meshes/base_plate.${mesh_format}"/>
       </geometry>
-      <material name="base_plate_5_material">
+      <material name="base_plate_bottom_left_material">
         <color rgba="0.117647 0.117647 0.117647 1"/>
       </material>
@@ -353,5 +353,5 @@
       </geometry>
     </collision>
-    <!-- Part base_plate_6 -->
+    <!-- Part base_plate_bottom_right -->
     <visual>
       <origin xyz="-0.0005 -0 0" rpy="0 -0 -1.5708"/>
@@ -359,5 +359,5 @@
         <mesh filename="package://bumperbot_description/meshes/base_plate.${mesh_format}"/>
       </geometry>
-      <material name="base_plate_6_material">
+      <material name="base_plate_bottom_right_material">
         <color rgba="0.117647 0.117647 0.117647 1"/>
       </material>
@@ -367,4 +367,30 @@
       <geometry>
         <mesh filename="package://bumperbot_description/meshes/base_plate.${mesh_format}"/>
+      </geometry>
+    </collision>
+    <!-- Part raspberry_pi_5 -->
+    <visual>
+      <origin xyz="0.025 0 0.046" rpy="0 0 1.5708"/>
+      <geometry>
+        <mesh filename="package://bumperbot_description/meshes/raspberry_pi_5.gltf"/>
+      </geometry>
+    </visual>
+    <collision>
+      <origin xyz="0.025 0 0.046" rpy="0 0 1.5708"/>
+      <geometry>
+        <mesh filename="package://bumperbot_description/meshes/raspberry_pi_5.gltf"/>
+      </geometry>
+    </collision>
+    <!-- Part l298n -->
+    <visual>
+      <origin xyz="-0.03 0 0.046" rpy="0 0 0"/>
+      <geometry>
+        <mesh filename="package://bumperbot_description/meshes/l298n.gltf"/>
+      </geometry>
+    </visual>
+    <collision>
+      <origin xyz="0.03 0 0.046" rpy="0 0 1.5708"/>
+      <geometry>
+        <mesh filename="package://bumperbot_description/meshes/l298n.gltf"/>
       </geometry>
     </collision>

Commit message: refactor: split base plate meshes and correct kinematic center alignment
- Replaced single base plate mesh with base_plate_left and base_plate_right halves
- Corrected misaligned base origin to eliminate asymmetric wheel separation
- Fixed slight physical tracking deviation to ensure absolute straight-line travel

File: src/Odometry_and_Control/bumperbot_description/urdf/include/bumperbot_mobile_base.xacro (robot description, xacro)
@@ -13,13 +13,13 @@
   <link name="base_link">
     <inertial>
-      <origin xyz="-0.000500099 3.9e-11 0.0388508" rpy="0 0 0"/>
+      <origin xyz="-9.8651e-08 -0 0.0388508" rpy="0 0 0"/>
       <mass value="0.427641"/>
-      <inertia ixx="0.000917472" ixy="-1.75126e-05" ixz="-6.25e-10" iyy="0.000910074" iyz="2e-12" izz="0.0011829"/>
+      <inertia ixx="0.000917472" ixy="-1.75126e-05" ixz="-6.26e-10" iyy="0.000910074" iyz="-0" izz="0.0011829"/>
     </inertial>
     <!-- Part spacer_hex -->
     <visual>
-      <origin xyz="0.0635 -0.024 0.0434998" rpy="0 -0 -0"/>
-      <geometry>
-        <mesh filename="package://bumperbot_description/meshes/spacer_hex.${mesh_format}"/>
+      <origin xyz="-0.064 0.024 0.0434998" rpy="0 -0 0"/>
+      <geometry>
+        <mesh filename="package://bumperbot_description/meshes/spacer_hex.gltf"/>
       </geometry>
       <material name="spacer_hex_material">
@@ -28,14 +28,14 @@
     </visual>
     <collision>
-      <origin xyz="0.0635 -0.024 0.0434998" rpy="0 -0 -0"/>
-      <geometry>
-        <mesh filename="package://bumperbot_description/meshes/spacer_hex.${mesh_format}"/>
+      <origin xyz="-0.064 0.024 0.0434998" rpy="0 -0 0"/>
+      <geometry>
+        <mesh filename="package://bumperbot_description/meshes/spacer_hex.gltf"/>
       </geometry>
     </collision>
     <!-- Part spacer_hex_2 -->
     <visual>
-      <origin xyz="-0.0645 -0.012 0.0434998" rpy="0 -0 -0"/>
-      <geometry>
-        <mesh filename="package://bumperbot_description/meshes/spacer_hex.${mesh_format}"/>
+      <origin xyz="0.024 0.064 0.0434998" rpy="0 -0 0.523599"/>
+      <geometry>
+        <mesh filename="package://bumperbot_description/meshes/spacer_hex.gltf"/>
       </geometry>
       <material name="spacer_hex_2_material">
@@ -44,14 +44,14 @@
     </visual>
     <collision>
-      <origin xyz="-0.0645 -0.012 0.0434998" rpy="0 -0 -0"/>
-      <geometry>
-        <mesh filename="package://bumperbot_description/meshes/spacer_hex.${mesh_format}"/>
+      <origin xyz="0.024 0.064 0.0434998" rpy="0 -0 0.523599"/>
+      <geometry>
+        <mesh filename="package://bumperbot_description/meshes/spacer_hex.gltf"/>
       </geometry>
     </collision>
     <!-- Part spacer_hex_3 -->
     <visual>
-      <origin xyz="0.0635 0.012 0.0434998" rpy="0 0 -0"/>
-      <geometry>
-        <mesh filename="package://bumperbot_description/meshes/spacer_hex.${mesh_format}"/>
+      <origin xyz="-0.064 -0.012 0.0434998" rpy="0 -0 0"/>
+      <geometry>
+        <mesh filename="package://bumperbot_description/meshes/spacer_hex.gltf"/>
       </geometry>
       <material name="spacer_hex_3_material">
@@ -60,14 +60,14 @@
     </visual>
     <collision>
-      <origin xyz="0.0635 0.012 0.0434998" rpy="0 0 -0"/>
-      <geometry>
-        <mesh filename="package://bumperbot_description/meshes/spacer_hex.${mesh_format}"/>
+      <origin xyz="-0.064 -0.012 0.0434998" rpy="0 -0 0"/>
+      <geometry>
+        <mesh filename="package://bumperbot_description/meshes/spacer_hex.gltf"/>
       </geometry>
     </collision>
     <!-- Part spacer_hex_4 -->
     <visual>
-      <origin xyz="0.0235 0.064 0.0434998" rpy="0 -0 -1.5708"/>
-      <geometry>
-        <mesh filename="package://bumperbot_description/meshes/spacer_hex.${mesh_format}"/>
+      <origin xyz="-0.024 -0.064 0.0434998" rpy="0 -0 0.523599"/>
+      <geometry>
+        <mesh filename="package://bumperbot_description/meshes/spacer_hex.gltf"/>
       </geometry>
       <material name="spacer_hex_4_material">
@@ -76,46 +76,46 @@
     </visual>
     <collision>
-      <origin xyz="0.0235 0.064 0.0434998" rpy="0 -0 -1.5708"/>
-      <geometry>
-        <mesh filename="package://bumperbot_description/meshes/spacer_hex.${mesh_format}"/>
-      </geometry>
-    </collision>
-    <!-- Part base_plate_mid_left -->
-    <visual>
-      <origin xyz="-0.0005 -0 0.037" rpy="0 -0 1.5708"/>
-      <geometry>
-        <mesh filename="package://bumperbot_description/meshes/base_plate.${mesh_format}"/>
-      </geometry>
-      <material name="base_plate_mid_left_material">
+      <origin xyz="-0.024 -0.064 0.0434998" rpy="0 -0 0.523599"/>
+      <geometry>
+        <mesh filename="package://bumperbot_description/meshes/spacer_hex.gltf"/>
+      </geometry>
+    </collision>
+    <!-- Part spacer_hex_5 -->
+    <visual>
+      <origin xyz="0.064 0.012 0.0434998" rpy="0 -0 0"/>
+      <geometry>
+        <mesh filename="package://bumperbot_description/meshes/spacer_hex.gltf"/>
+      </geometry>
+      <material name="spacer_hex_5_material">
+        <color rgba="0.980392 0.796078 0.262745 1"/>
+      </material>
+    </visual>
+    <collision>
+      <origin xyz="0.064 0.012 0.0434998" rpy="0 -0 0"/>
+      <geometry>
+        <mesh filename="package://bumperbot_description/meshes/spacer_hex.gltf"/>
+      </geometry>
+    </collision>
+    <!-- Part base_plate_right -->
+    <visual>
+      <origin xyz="0 0 0.037" rpy="0 -0 0"/>
+      <geometry>
+        <mesh filename="package://bumperbot_description/meshes/base_plate_right.gltf"/>
+      </geometry>
+      <material name="base_plate_right_material">
         <color rgba="0.117647 0.117647 0.117647 1"/>
       </material>
     </visual>
     <collision>
-      <origin xyz="-0.0005 -0 0.037" rpy="0 -0 1.5708"/>
-      <geometry>
-        <mesh filename="package://bumperbot_description/meshes/base_plate.${mesh_format}"/>
-      </geometry>
-    </collision>
-    <!-- Part spacer_hex_5 -->
-    <visual>
-      <origin xyz="-0.0645 0.024 0.0434998" rpy="-0 -0 -0"/>
-      <geometry>
-        <mesh filename="package://bumperbot_description/meshes/spacer_hex.${mesh_format}"/>
-      </geometry>
-      <material name="spacer_hex_5_material">
-        <color rgba="0.980392 0.796078 0.262745 1"/>
-      </material>
-    </visual>
-    <collision>
-      <origin xyz="-0.0645 0.024 0.0434998" rpy="-0 -0 -0"/>
-      <geometry>
-        <mesh filename="package://bumperbot_description/meshes/spacer_hex.${mesh_format}"/>
+      <origin xyz="0 0 0.037" rpy="0 -0 0"/>
+      <geometry>
+        <mesh filename="package://bumperbot_description/meshes/base_plate_right.gltf"/>
       </geometry>
     </collision>
     <!-- Part spacer_hex_6 -->
     <visual>
-      <origin xyz="-0.0245 -0.064 0.0434998" rpy="0 -0 1.5708"/>
-      <geometry>
-        <mesh filename="package://bumperbot_description/meshes/spacer_hex.${mesh_format}"/>
+      <origin xyz="0.064 -0.024 0.0434998" rpy="0 -0 0"/>
+      <geometry>
+        <mesh filename="package://bumperbot_description/meshes/spacer_hex.gltf"/>
       </geometry>
       <material name="spacer_hex_6_material">
@@ -124,62 +124,62 @@
     </visual>
     <collision>
-      <origin xyz="-0.0245 -0.064 0.0434998" rpy="0 -0 1.5708"/>
-      <geometry>
-        <mesh filename="package://bumperbot_description/meshes/spacer_hex.${mesh_format}"/>
-      </geometry>
-    </collision>
-    <!-- Part base_plate_mid_right -->
-    <visual>
-      <origin xyz="-0.0005 -0 0.037" rpy="0 -0 -1.5708"/>
-      <geometry>
-        <mesh filename="package://bumperbot_description/meshes/base_plate.${mesh_format}"/>
-      </geometry>
-      <material name="base_plate_mid_right_material">
+      <origin xyz="0.064 -0.024 0.0434998" rpy="0 -0 0"/>
+      <geometry>
+        <mesh filename="package://bumperbot_description/meshes/spacer_hex.gltf"/>
+      </geometry>
+    </collision>
+    <!-- Part base_plate_left -->
+    <visual>
+      <origin xyz="0 0 0.037" rpy="0 -0 0"/>
+      <geometry>
+        <mesh filename="package://bumperbot_description/meshes/base_plate_left.gltf"/>
+      </geometry>
+      <material name="base_plate_left_material">
         <color rgba="0.117647 0.117647 0.117647 1"/>
       </material>
     </visual>
     <collision>
-      <origin xyz="-0.0005 -0 0.037" rpy="0 -0 -1.5708"/>
-      <geometry>
-        <mesh filename="package://bumperbot_description/meshes/base_plate.${mesh_format}"/>
-      </geometry>
-    </collision>
-    <!-- Part base_plate_top_left -->
-    <visual>
-      <origin xyz="-0.0005 -0 0.074" rpy="0 -0 1.5708"/>
-      <geometry>
-        <mesh filename="package://bumperbot_description/meshes/base_plate.${mesh_format}"/>
-      </geometry>
-      <material name="base_plate_top_left_material">
+      <origin xyz="0 0 0.037" rpy="0 -0 0"/>
+      <geometry>
+        <mesh filename="package://bumperbot_description/meshes/base_plate_left.gltf"/>
+      </geometry>
+    </collision>
+    <!-- Part base_plate_right_2 -->
+    <visual>
+      <origin xyz="0 0 0.074" rpy="0 -0 0"/>
+      <geometry>
+        <mesh filename="package://bumperbot_description/meshes/base_plate_right.gltf"/>
+      </geometry>
+      <material name="base_plate_right_2_material">
         <color rgba="0.117647 0.117647 0.117647 1"/>
       </material>
     </visual>
     <collision>
-      <origin xyz="-0.0005 -0 0.074" rpy="0 -0 1.5708"/>
-      <geometry>
-        <mesh filename="package://bumperbot_description/meshes/base_plate.${mesh_format}"/>
-      </geometry>
-    </collision>
-    <!-- Part base_plate_top_right -->
-    <visual>
-      <origin xyz="-0.0005 -0 0.074" rpy="0 -0 -1.5708"/>
-      <geometry>
-        <mesh filename="package://bumperbot_description/meshes/base_plate.${mesh_format}"/>
-      </geometry>
-      <material name="base_plate_top_right_material">
+      <origin xyz="0 0 0.074" rpy="0 -0 0"/>
+      <geometry>
+        <mesh filename="package://bumperbot_description/meshes/base_plate_right.gltf"/>
+      </geometry>
+    </collision>
+    <!-- Part base_plate_left_2 -->
+    <visual>
+      <origin xyz="0 0 0.074" rpy="0 -0 0"/>
+      <geometry>
+        <mesh filename="package://bumperbot_description/meshes/base_plate_left.gltf"/>
+      </geometry>
+      <material name="base_plate_left_2_material">
         <color rgba="0.117647 0.117647 0.117647 1"/>
       </material>
     </visual>
     <collision>
-      <origin xyz="-0.0005 -0 0.074" rpy="0 -0 -1.5708"/>
-      <geometry>
-        <mesh filename="package://bumperbot_description/meshes/base_plate.${mesh_format}"/>
+      <origin xyz="0 0 0.074" rpy="0 -0 0"/>
+      <geometry>
+        <mesh filename="package://bumperbot_description/meshes/base_plate_left.gltf"/>
       </geometry>
     </collision>
     <!-- Part spacer_hex_7 -->
     <visual>
-      <origin xyz="0.0635 -0.024 0.0064998" rpy="0 -0 0"/>
-      <geometry>
-        <mesh filename="package://bumperbot_description/meshes/spacer_hex.${mesh_format}"/>
+      <origin xyz="-0.064 0.024 0.0064998" rpy="0 -0 0"/>
+      <geometry>
+        <mesh filename="package://bumperbot_description/meshes/spacer_hex.gltf"/>
       </geometry>
       <material name="spacer_hex_7_material">
@@ -188,14 +188,14 @@
     </visual>
     <collision>
-      <origin xyz="0.0635 -0.024 0.0064998" rpy="0 -0 0"/>
-      <geometry>
-        <mesh filename="package://bumperbot_description/meshes/spacer_hex.${mesh_format}"/>
+      <origin xyz="-0.064 0.024 0.0064998" rpy="0 -0 0"/>
+      <geometry>
+        <mesh filename="package://bumperbot_description/meshes/spacer_hex.gltf"/>
       </geometry>
     </collision>
     <!-- Part motor_bracket_left -->
     <visual>
-      <origin xyz="-0.0005 0.0482736 0.00899984" rpy="0 -0 0"/>
-      <geometry>
-        <mesh filename="package://bumperbot_description/meshes/motor_bracket_left.${mesh_format}"/>
+      <origin xyz="0 0.0482736 0.0089998" rpy="0 -0 0"/>
+      <geometry>
+        <mesh filename="package://bumperbot_description/meshes/motor_bracket_left.gltf"/>
       </geometry>
       <material name="motor_bracket_left_material">
@@ -204,62 +204,14 @@
     </visual>
     <collision>
-      <origin xyz="-0.0005 0.0482736 0.00899984" rpy="0 -0 0"/>
-      <geometry>
-        <mesh filename="package://bumperbot_description/meshes/motor_bracket_left.${mesh_format}"/>
-      </geometry>
-    </collision>
-    <!-- Part spacer_hex_8 -->
-    <visual>
-      <origin xyz="-0.0645 -0.012 0.0064998" rpy="0 -0 0"/>
-      <geometry>
-        <mesh filename="package://bumperbot_description/meshes/spacer_hex.${mesh_format}"/>
-      </geometry>
-      <material name="spacer_hex_8_material">
-        <color rgba="0.980392 0.796078 0.262745 1"/>
-      </material>
-    </visual>
-    <collision>
-      <origin xyz="-0.0645 -0.012 0.0064998" rpy="0 -0 0"/>
-      <geometry>
-        <mesh filename="package://bumperbot_description/meshes/spacer_hex.${mesh_format}"/>
-      </geometry>
-    </collision>
-    <!-- Part spacer_hex_9 -->
-    <visual>
-      <origin xyz="0.0635 0.012 0.0064998" rpy="0 0 0"/>
-      <geometry>
-        <mesh filename="package://bumperbot_description/meshes/spacer_hex.${mesh_format}"/>
-      </geometry>
-      <material name="spacer_hex_9_material">
-        <color rgba="0.980392 0.796078 0.262745 1"/>
-      </material>
-    </visual>
-    <collision>
-      <origin xyz="0.0635 0.012 0.0064998" rpy="0 0 0"/>
-      <geometry>
-        <mesh filename="package://bumperbot_description/meshes/spacer_hex.${mesh_format}"/>
-      </geometry>
-    </collision>
-    <!-- Part spacer_hex_10 -->
-    <visual>
-      <origin xyz="0.0235 0.064 0.0064998" rpy="0 -0 -1.5708"/>
-      <geometry>
-        <mesh filename="package://bumperbot_description/meshes/spacer_hex.${mesh_format}"/>
-      </geometry>
-      <material name="spacer_hex_10_material">
-        <color rgba="0.980392 0.796078 0.262745 1"/>
-      </material>
-    </visual>
-    <collision>
-      <origin xyz="0.0235 0.064 0.0064998" rpy="0 -0 -1.5708"/>
-      <geometry>
-        <mesh filename="package://bumperbot_description/meshes/spacer_hex.${mesh_format}"/>
+      <origin xyz="0 0.0482736 0.0089998" rpy="0 -0 0"/>
+      <geometry>
+        <mesh filename="package://bumperbot_description/meshes/motor_bracket_left.gltf"/>
       </geometry>
     </collision>
     <!-- Part motor_bracket_right -->
     <visual>
-      <origin xyz="-0.0005 -0.0482736 0.00899984" rpy="0 -0 0"/>
-      <geometry>
-        <mesh filename="package://bumperbot_description/meshes/motor_bracket_right.${mesh_format}"/>
+      <origin xyz="-0 -0.0482736 0.0089998" rpy="0 -0 0"/>
+      <geometry>
+        <mesh filename="package://bumperbot_description/meshes/motor_bracket_right.gltf"/>
       </geometry>
       <material name="motor_bracket_right_material">
@@ -268,14 +220,14 @@
     </visual>
     <collision>
-      <origin xyz="-0.0005 -0.0482736 0.00899984" rpy="0 -0 0"/>
-      <geometry>
-        <mesh filename="package://bumperbot_description/meshes/motor_bracket_right.${mesh_format}"/>
+      <origin xyz="-0 -0.0482736 0.0089998" rpy="0 -0 0"/>
+      <geometry>
+        <mesh filename="package://bumperbot_description/meshes/motor_bracket_right.gltf"/>
       </geometry>
     </collision>
     <!-- Part actuatordc_left -->
     <visual>
-      <origin xyz="-0.0005 0.0667736 0.0239998" rpy="-0 -0 0"/>
-      <geometry>
-        <mesh filename="package://bumperbot_description/meshes/actuatordc_left.${mesh_format}"/>
+      <origin xyz="0 0.0667736 0.0239998" rpy="0 -0 0"/>
+      <geometry>
+        <mesh filename="package://bumperbot_description/meshes/actuatordc_left.gltf"/>
       </geometry>
       <material name="actuatordc_left_material">
@@ -284,30 +236,30 @@
     </visual>
     <collision>
-      <origin xyz="-0.0005 0.0667736 0.0239998" rpy="-0 -0 0"/>
-      <geometry>
-        <mesh filename="package://bumperbot_description/meshes/actuatordc_left.${mesh_format}"/>
-      </geometry>
-    </collision>
-    <!-- Part base_plate_bottom_left -->
-    <visual>
-      <origin xyz="-0.0005 -0 0" rpy="0 -0 1.5708"/>
-      <geometry>
-        <mesh filename="package://bumperbot_description/meshes/base_plate.${mesh_format}"/>
-      </geometry>
-      <material name="base_plate_bottom_left_material">
-        <color rgba="0.117647 0.117647 0.117647 1"/>
-      </material>
-    </visual>
-    <collision>
-      <origin xyz="-0.0005 -0 0" rpy="0 -0 1.5708"/>
-      <geometry>
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