Commit message: refactor: relocate caster_z_offset property to robot_properties.xacro for centralized configuration

File: src/Odometry_and_Control/bumperbot_description/urdf/include/bumperbot_mobile_base.xacro (robot description, xacro)
@@ -1,6 +1,4 @@
 <?xml version="1.0" ?>
 <robot xmlns:xacro="http://ros.org/wiki/xacro">
-  <xacro:property name="caster_z_offset" value="-0.005237682" />
-<!-- -0.005237682 -->
   <link name="base_footprint"/>
   <joint name="base_footprint_joint" type="fixed">

File: src/Odometry_and_Control/bumperbot_description/urdf/include/robot_properties.xacro (robot description, xacro)
@@ -6,4 +6,5 @@
   <xacro:property name="base_height" value="0.083" />
   <xacro:property name="base_mass" value="0.5" />
+  <xacro:property name="caster_z_offset" value="-0.005237682" />
   <xacro:property name="caster_radius" value="0.005" />
   <xacro:property name="caster_mass" value="0.02" />
