Commit message: chore: update base_footprint_to_base_link_z to 0.01 for precision alignment

File: src/Odometry_and_Control/bumperbot_description/urdf/include/robot_properties.xacro (robot description, xacro)
@@ -1,5 +1,5 @@
 <?xml version="1.0" ?>
 <robot xmlns:xacro="http://ros.org/wiki/xacro">
-  <xacro:property name="base_footprint_to_base_link_z" value="0.00999676" />
+  <xacro:property name="base_footprint_to_base_link_z" value="0.01" />
   <xacro:property name="base_length" value="0.13763785" />
   <xacro:property name="base_width" value="0.13763785" />
